Commit message: modified for navigation

File: urdf/includes/gazebo/inertias.xacro (robot description, xacro)
@@ -44,3 +44,13 @@
   </xacro:macro>
   <!-- cylinder inertia -->
+  <!-- open cylinder inertia -->
+  <xacro:macro name="cylinder_inertia" params="mass r1 r2 h">
+    <inertial>
+      <mass value="${mass}"/>
+      <inertia  ixx="${mass*(3*(r1*r1 + r2*r2)+h*h)/12}" ixy = "0" ixz = "0"
+                iyy="${mass*(3*(r1*r1 + r2*r2)+h*h)/12}" iyz = "0"
+                izz="${mass*(r1*r1 + r2*r2)/2}" />
+    </inertial>
+  </xacro:macro>
+  <!-- open cylinder inertia -->
 </robot>

File: urdf/includes/parts/wheels/wheel.xacro (robot description, xacro)
@@ -8,10 +8,7 @@
   <xacro:property name="wheelc_len" value="0.015" />
   <xacro:property name="wheelc_r" value = "0.026" />
-  <xacro:property name="wheel_shaft_mass" value = "0.0028" />
-  <xacro:property name="wheelc_mass" value = "0.0272" />
-  <xacro:property name="wheel_mass" value = "0.0181" />
-  <!--xacro:property name="wheel_shaft_mass" value="0.6" />
-  <xacro:property name="wheelc_mass" value="0.6" />
-  <xacro:property name="wheel_mass" value="0.6" /-->
+ <xacro:property name="wheel_shaft_mass" value = "0.000283495" /> <!--0.000283495 0.0028 -->
+  <xacro:property name="wheelc_mass" value = "0.283495" />  <!--0.283495 0.00283495 0.0272 -->
+  <xacro:property name="wheel_mass" value = "3.0" />         <!--2.5 0.0181 -->
   <!-- Wheel constants -->
   <!-- Inertia Macro -->
@@ -56,6 +53,6 @@
       </geometry>
     </collision>
-    <xacro:inertia mass="0.6" />
-    <!--xacro:cylinder_inertia mass="${wheelc_mass}" r="${wheelc_r}" h="${wheelc_len}" /-->
+    <!--xacro:inertia mass="0.6" /-->
+    <xacro:cylinder_inertia mass="${wheelc_mass}" r="${wheelc_r}" h="${wheelc_len}" />
   </link>
   <joint name="${prefix}_shaft_wheelc_joint" type="fixed">
@@ -78,6 +75,6 @@
       </geometry>
     </collision>
-    <xacro:inertia mass="0.6"/>
-    <!--xacro:cylinder_inertia mass="${wheel_mass}" r="${wheelc_r + 0.0065}" h="${wheelc_len}" /-->
+    <!--xacro:inertia mass="0.6"/-->
+    <xacro:open_cylinder_inertia mass="${wheel_mass}" r1="${wheelc_r}" r2="${wheelc_r + 0.0065}" h="${wheelc_len}" />
   </link>
   <joint name="${prefix}_wheel_joint" type="continuous">

Commit message: fixed bug of previous commit

File: urdf/includes/gazebo/inertias.xacro (robot description, xacro)
@@ -45,5 +45,5 @@
   <!-- cylinder inertia -->
   <!-- open cylinder inertia -->
-  <xacro:macro name="cylinder_inertia" params="mass r1 r2 h">
+  <xacro:macro name="open_cylinder_inertia" params="mass r1 r2 h">
     <inertial>
       <mass value="${mass}"/>

File: urdf/includes/parts/wheels/wheel.xacro (robot description, xacro)
@@ -8,7 +8,7 @@
   <xacro:property name="wheelc_len" value="0.015" />
   <xacro:property name="wheelc_r" value = "0.026" />
- <xacro:property name="wheel_shaft_mass" value = "0.000283495" /> <!--0.000283495 0.0028 -->
+  <xacro:property name="wheel_shaft_mass" value = "0.000283495" /> <!--0.000283495 0.0028 -->
   <xacro:property name="wheelc_mass" value = "0.283495" />  <!--0.283495 0.00283495 0.0272 -->
-  <xacro:property name="wheel_mass" value = "3.0" />         <!--2.5 0.0181 -->
+  <xacro:property name="wheel_mass" value = "0.0181" />         <!--3.0 0.0181 -->
   <!-- Wheel constants -->
   <!-- Inertia Macro -->
@@ -53,6 +53,6 @@
       </geometry>
     </collision>
-    <!--xacro:inertia mass="0.6" /-->
-    <xacro:cylinder_inertia mass="${wheelc_mass}" r="${wheelc_r}" h="${wheelc_len}" />
+    <xacro:inertia mass="0.6" />
+    <!--xacro:cylinder_inertia mass="${wheelc_mass}" r="${wheelc_r}" h="${wheelc_len}" /-->
   </link>
   <joint name="${prefix}_shaft_wheelc_joint" type="fixed">
@@ -75,6 +75,6 @@
       </geometry>
     </collision>
-    <!--xacro:inertia mass="0.6"/-->
-    <xacro:open_cylinder_inertia mass="${wheel_mass}" r1="${wheelc_r}" r2="${wheelc_r + 0.0065}" h="${wheelc_len}" />
+    <xacro:inertia mass="0.6"/>
+    <!--xacro:open_cylinder_inertia mass="${wheel_mass}" r1="${wheelc_r}" r2="${wheelc_r + 0.0065}" h="${wheelc_len}" /-->
   </link>
   <joint name="${prefix}_wheel_joint" type="continuous">
