Commit message: changed imu names to standard names like imu_link

File: urdf/includes/gazebo/imu.gazebo.xacro (robot description, xacro)
@@ -6,5 +6,5 @@
         <plugin name="${imu_name}_plugin" filename="libhector_gazebo_ros_imu.so">
           <alwaysOn>true</alwaysOn>
-          <bodyName>${imu_name}_base</bodyName>
+          <bodyName>${imu_name}_link</bodyName>
           <topicName>${topic_ns}</topicName>
           <serviceName>${topic_ns}_service</serviceName>
@@ -13,4 +13,32 @@
         </plugin>
       </gazebo>
+  <!--gazebo>
+    <plugin name="${imu_name}_plugin" filename="libgazebo_ros_imu.so">
+      <alwaysOn>true</alwaysOn>
+      <bodyName>${imu_name}_link</bodyName>
+      <frameName>${imu_name}_link</frameName>
+      <topicName>${topic_ns}</topicName>
+      <serviceName>${topic_ns}_service</serviceName>
+      <gaussianNoise>0.0</gaussianNoise>
+      <updateRate>200</updateRate>
+      <imu>
+        <noise>
+          <type>gaussian</type>
+          <rate>
+            <mean>0.0</mean>
+            <stddev>2e-4</stddev>
+            <bias_mean>0.0000075</bias_mean>
+            <bias_stddev>0.0000008</bias_stddev>
+          </rate>
+          <accel>
+            <mean>0.0</mean>
+            <stddev>1.7e-2</stddev>
+            <bias_mean>0.1</bias_mean>
+            <bias_stddev>0.001</bias_stddev>
+          </accel>
+        </noise>
+      </imu>
+    </plugin>
+  </gazebo-->
   </xacro:macro>
 </robot>

File: urdf/includes/gazebo/jetbot.gazebo.xacro (robot description, xacro)
@@ -166,5 +166,5 @@
     <material>Gazebo/GreenTransparent</material>
   </gazebo>
-  <gazebo reference="bno055_base">
+  <gazebo reference="imu_link">
     <material>Gazebo/Yellow</material>
   </gazebo>

File: urdf/includes/parts/sensors/imu/bno055.urdf.xacro (robot description, xacro)
@@ -12,11 +12,11 @@
   <xacro:include filename="$(find jetbot_description)/urdf/includes/gazebo/imu.gazebo.xacro" />
   <!-- IMU BNO055 -->
-  <xacro:macro name="sensor_imu" params="name topic_ns:=bno055 parent *origin">
+  <xacro:macro name="sensor_imu" params="name topic_ns:=imu parent *origin">
     <joint name="{name}_joint" type="fixed">
       <parent link="${parent}"/>
-      <child link="${name}_base"/>
+      <child link="${name}_link"/>
       <xacro:insert_block name="origin" />
     </joint>
-    <link name="${name}_base">
+    <link name="${name}_link">
       <visual>
         <origin xyz="-${bno_width/2} ${bno_height/2} 0" rpy="${pi/2} 0 0"/>

File: urdf/jetbot.urdf.xacro (robot description, xacro)
@@ -50,5 +50,5 @@
   <!-- IMU -->
   <xacro:if value="$(arg imu_enable)" >
-    <xacro:sensor_imu name="bno055" topic_ns="bno_imu" parent="pcb_boards" >
+    <xacro:sensor_imu name="imu" topic_ns="imu" parent="pcb_boards" >
       <origin xyz="0 0 0.0275" rpy="0 0 0" />
     </xacro:sensor_imu>
@@ -56,5 +56,5 @@
   <!-- GPS -->
   <xacro:if value="$(arg gps_enable)" >
-    <xacro:sensor_gps name="mtk3339" topic_ns="mtk_gps" parent="bno055_base" >
+    <xacro:sensor_gps name="mtk3339" topic_ns="mtk_gps" parent="imu_link" >
       <origin xyz="-0.044 0 0" rpy="0 0 0" />
     </xacro:sensor_gps>
